File: kicad/Programmer-20K-ESP/Programmer-20K-ESP.kicad_pcb (KiCad board)
At the start: 2 copper layers, 62.3 x 32.9 mm, 18 parts, among them J1 Conn_01x08, J2 USB_C_Receptacle_PowerOnly_6P, J3 Programmer, SW1 ESP_RESET, SW2 STATUS, U1 ESP32-WROVER-B, U2 AMS1117-3.3

Commit message: Support for WS2812B RGB LED
Parts:
- added C6: 100n, Capacitor_SMD:C_0805_2012Metric_Pad1.18x1.45mm_HandSolder, F.Cu at (117.4, 75.6)
- added R5: 5K1, Resistor_SMD:R_0805_2012Metric_Pad1.20x1.40mm_HandSolder, F.Cu at (93.4, 81.0)
- added R6: 5K1, Resistor_SMD:R_0805_2012Metric_Pad1.20x1.40mm_HandSolder, F.Cu at (93.4, 78.8)
Connections:
- J2 pad A5: unconnected-(J2-CC1-PadA5) -> Net-(J2-CC1)
- J2 pad B5: unconnected-(J2-CC2-PadB5) -> Net-(J2-CC2)
- J2 pad S1: unconnected-(J2-SHIELD-PadS1)_1 -> GND
Routing:
- net Net-(J2-CC2): track 0.00 -> 9.92 mm
- net Net-(J2-CC1): track 0.00 -> 8.52 mm
- net GND: track 63.5 -> 66.9 mm, vias 13 -> 15
- net LED: track 37.0 -> 38.4 mm
- net +5V: track 75.9 -> 77.2 mm
